File: GORAT circuit diagram/GORAT circuit diagram.kicad_pcb (KiCad board)
At the start: 2 copper layers, 108.5 x 71.5 mm, 77 parts, among them J1 AudioJack2, J2 AudioJack2, J3 Conn_01x08_Socket, J4 Conn_01x08_Socket, J6 Barrel_Jack, J8 Conn_01x02_Socket, J9 Conn_01x02_Socket, Q1 J111, SW1 SW_DPDT_x2, SW8 SW_Rotary2x6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

Commit message: update board and layout
Parts:
- removed SP3, SP4: Conn_01x02_Socket, Connector_PinHeader_2.54mm:PinHeader_1x02_P2.54mm_Vertical
- added C6: 1u, Capacitor_THT:C_Disc_D4.7mm_W2.5mm_P5.00mm, B.Cu at (127.5, 84.5)
- added R27: 47k, Resistor_THT:R_Axial_DIN0207_L6.3mm_D2.5mm_P10.16mm_Horizontal, B.Cu at (137.6, 88.5)
- R15: value 100k -> 10k
- R26: moved to B.Cu
- moved R2 22.9 mm to (169.2, 82.7), turned to -90 degrees
- moved R25 15.6 mm to (166.0, 92.8), turned to 90 degrees
- moved R1 14.6 mm to (192.1, 81.0)
- moved R24 14.6 mm to (192.1, 84.2)
- moved R10 14.5 mm to (192.1, 90.8)
- moved R7 14.5 mm to (181.9, 87.5)
- moved C1 14.4 mm to (177.8, 89.5)
- moved C18 14.4 mm to (172.8, 86.2)
- moved C5 14.4 mm to (172.8, 83.0)
- moved R22 10.3 mm to (87.2, 89.4), turned to -90 degrees
- moved C12 9.10 mm to (172.8, 92.8), turned to 0 degrees
- moved D3 8.90 mm to (166.8, 97.9), turned to -90 degrees
- moved C8 8.39 mm to (144.8, 100.8), turned to 180 degrees
- moved R23 7.93 mm to (97.3, 83.0), turned to 180 degrees
- moved C4 6.62 mm to (139.8, 124.5), turned to 0 degrees
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- renumbered RV4-BLEND2 to RV2-TILT1
Connections:
- R16 pad 2: Net-(U3A-+) -> Net-(C6-Pad1)
- R17 pad 2: Net-(U3A-+) -> Net-(C6-Pad1)
Routing:
- net +9V: track 0.00 -> 110.0 mm
- net +4.5V: track 0.00 -> 108.0 mm, vias 0 -> 1
- net Net-(SW1B-C): track 0.00 -> 101.6 mm
- net /JackOut1: track 0.00 -> 100.9 mm, vias 0 -> 1
- net Net-(SW1A-C): track 0.00 -> 89.0 mm
- net Net-(U2A--): track 0.00 -> 79.0 mm
- net Net-(SW1A-A): track 0.00 -> 68.3 mm
- net Vin1: track 0.00 -> 66.1 mm, vias 0 -> 1
- net /+9v Jack1: track 0.00 -> 61.0 mm, vias 0 -> 1
- net Net-(C23-Pad1): track 0.00 -> 56.2 mm, vias 0 -> 1
- net Net-(D5-K): track 0.00 -> 50.5 mm
- net Net-(C3-Pad2): track 0.00 -> 49.9 mm
- net Net-(D7-K): track 0.00 -> 47.0 mm, vias 0 -> 1
- net Net-(R17-Pad1): track 0.00 -> 46.4 mm, vias 0 -> 1
- net Net-(D1-K): track 0.00 -> 45.3 mm
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Other:
- outline, holes or cut-outs redrawn

Commit message: Update KiCad files: remap nets and rename caps
Synchronise PCB and schematic: remap many net indices across GORAT circuit diagram (.kicad_pcb, .kicad_sch, .kicad_prl, .kicad_pro) to match the schematic, and rename several capacitor references (e.g. C7/C15/C19 -> Cp7/Cp15/Cp19). Add autosave and CSV export files, update GoRAT spreadsheet, and refresh backup ZIPs (deleted older backups, added new ones). These changes ensure net and reference consistency between schematic and board files.
Parts:
- renumbered C11 to Cp11, C13 to Cp13, C14 to Cp14, C15 to Cp15, C19 to Cp19, C7 to Cp7
