File: GORAT circuit diagram/GORAT circuit diagram.kicad_pcb (KiCad board)
At the start: 2 copper layers, 108.5 x 71.5 mm, 77 parts, among them J1 AudioJack2, J2 AudioJack2, J3 Conn_01x08_Socket, J4 Conn_01x08_Socket, J6 Barrel_Jack, J8 Conn_01x02_Socket, J9 Conn_01x02_Socket, Q1 J111, SW1 SW_DPDT_x2, SW8 SW_Rotary2x6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

Commit message: V0.2 finished
Parts:
- moved D6 0.25 mm to (119.0, 130.8)
Connections:
- D7 pad 1: Net-(D7-K) -> Net-(D1-K)
- J8 pad 2: Net-(J8-Pin_1) -> Net-(J8-Pin_2)
- SW1 pad 2: Net-(J8-Pin_1) -> Net-(J8-Pin_2)
- SW8 pad 1: Net-(D2-A) -> Net-(D8-A)
- SW8 pad 2: Net-(D2-A) -> Net-(D8-A)
- SW8 pad 3: Net-(D8-A) -> Net-(D2-A)
- SW8 pad 4: Net-(D8-A) -> Net-(D2-A)
- SW8 pad 8: Net-(D7-K) -> Net-(SW8-Pad8)
- SW8 pad 9: Net-(D7-K) -> Net-(SW8-Pad8)
Routing:
- net Net-(D7-K): track 47.0 -> 0.00 mm, vias 1 -> 0
- net Net-(J8-Pin_2): track 0.00 -> 19.3 mm
- net Net-(R16-Pad1): track 8.81 -> 18.4 mm
- net Net-(D1-K): track 45.3 -> 52.0 mm
- net Net-(SW8-Pad8): track 0.00 -> 5.75 mm
- net Net-(D8-A): track 15.7 -> 20.6 mm
- net Net-(D5-K): track 50.5 -> 46.0 mm
- net Net-(J9-Pin_2): track 31.1 -> 26.7 mm
- net Net-(D2-A): track 16.8 -> 13.4 mm
- net +9V: track 110.0 -> 112.4 mm
- net Net-(J8-Pin_1): track 27.0 -> 28.5 mm
- net Net-(SW1A-C): track 89.0 -> 89.9 mm
- net Net-(C23-Pad1): track 56.2 -> 57.0 mm
Other:
- board text added: "GoRAT Distortion V0.2"
- board text removed: "GoRAT Distortion V1.2"
