File: GORAT circuit diagram/GORAT circuit diagram.kicad_pcb (KiCad board)
At the start: 2 copper layers, 108.5 x 71.5 mm, 77 parts, among them J1 AudioJack2, J2 AudioJack2, J3 Conn_01x08_Socket, J4 Conn_01x08_Socket, J6 Barrel_Jack, J8 Conn_01x02_Socket, J9 Conn_01x02_Socket, Q1 J111, SW1 SW_DPDT_x2, SW8 SW_Rotary2x6, U1 OP07CP, U2 TL072ACP, U3 TL072ACP

Commit message: Fixed pop by enabling always-on
Connections:
- D4 pad 2: Vin1 -> LED1
- J3 pad 6: /+9v Jack1 -> Vin1
- J3 pad 7: Vin1 -> LED1
- J4 pad 6: /+9v Jack2 -> Vin2
- J4 pad 7: Vin2 -> LED2
- J6 pad 1: /+9v Jack1 -> Vin1
- S1 pad P$7: /+9v Jack2 -> Vin2
- S1 pad P$8: Vin2 -> LED2
Routing:
- net /+9v Jack1: track 61.0 -> 0.00 mm, vias 1 -> 0
- net LED1: track 0.00 -> 31.0 mm
- net Vin1: track 66.1 -> 89.5 mm, vias 1 -> 2
- net /+9v Jack2: track 18.8 -> 0.00 mm
- net LED2: track 0.00 -> 15.5 mm
- net Vin2: track 14.5 -> 28.2 mm
- net SigOut1: vias 0 -> 1
Other:
- board text added: "GoRAT Distortion V0.3"
- board text removed: "GoRAT Distortion V0.2"
