File: GORAT circuit diagram/GORAT circuit diagram.kicad_sch (KiCad schematic)
At the start: 77 parts, among them J1 AudioJack2, J2 AudioJack2, J3 Conn_01x08_Socket, J4 Conn_01x08_Socket, J6 Barrel_Jack, J8 Conn_01x02_Socket, J9 Conn_01x02_Socket, Q1 J111, SW1 SW_DPDT_x2, SW8 SW_Rotary2x6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

Commit message: update
Other:
- note added: "Might be very low consider changing on test"
- note added: "change this, no need to use both lugs"
- note added: "consider increasing this if output is too low or decreasing it output too hot"
- note added: "perhaps no longer necessary, or reduce to like 1kohm? this section could go to virtual ground and remove some complexity"
- note added: "this is wrong fix it before next batch"
