File: GORAT circuit diagram/GORAT circuit diagram.kicad_sch (KiCad schematic)
At the start: 77 parts, among them J1 AudioJack2, J2 AudioJack2, J3 Conn_01x08_Socket, J4 Conn_01x08_Socket, J6 Barrel_Jack, J8 Conn_01x02_Socket, J9 Conn_01x02_Socket, Q1 J111, SW1 SW_DPDT_x2, SW8 SW_Rotary2x6, U1 OP07CP, U2 TL072ACP, U3 TL072ACP

Commit message: Fixed pop by enabling always-on
Connections:
- net +9v Jack1 is gone; now on net Vin1: J3.6 (Pin_6), J6.1
- net +9v Jack2 is gone; now on net Vin2: J4.6 (Pin_6), S1.P$7 (O)
- net Vin1: no longer D4.2 (A), J3.7 (Pin_7)
- net Vin2: no longer J4.7 (Pin_7), S1.P$8 (P)
- new net LED1: D4.2 (A), J3.7 (Pin_7)
- new net LED2: J4.7 (Pin_7), S1.P$8 (P)
Other:
- moved on the sheet: D4, R13
